File: hardware/StompFork/StompFork.kicad_sch (KiCad schematic)
At the start: 34 parts, among them J1 Line-Level Input, J2 Direct Output, J3 Stompbox Output 1, J4 Stompbox Output 2, J5 Power, U1 TL074

Commit message: Update comments
Other:
- note added: "Electrolytic or Film (PP/PET)"
- note added: "Polarized or Bipolar (C5-C7)"
- note added: "VGND is buffered mid‑rail. Do NOT connect to jack sleeves or chassis!"
Changed lines of the file:
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@@
 		(comment 3 "Active OpAmp audio signal splitter to feed multiple parallel stompboxes.")
 	)
+	(text "Electrolytic or Film (PP/PET)"
+		(exclude_from_sim no)
+		(at 52.324 31.242 0)
+		(effects
+			(font
+				(size 1.27 1.27)
+			)
+		)
+	)
+	(text "VGND is buffered mid‑rail.\nDo NOT connect to jack sleeves or chassis!"
+		(exclude_from_sim no)
+		(at 101.6 190.5 0)
+		(effects
+			(font
+				(size 1.27 1.27)
+			)
+		)
+	)
+	(text "Polarized or Bipolar (C5-C7)"
+		(exclude_from_sim no)
+		(at 238.252 31.242 0)
+		(effects
+			(font
+				(size 1.27 1.27)
+			)
+		)
+	)
 	(junction
 		(at 44.45 101.6)
@@
 			)
 		)
-		(property "Description" "Electrolytic or Film (PP/PET)"
+		(property "Description" "Polarized capacitor"
 			(at 52.324 29.718 90)
 			(effects
@@
 					(size 1.27 1.27)
 				)
+				(hide yes)
 			)
 		)
@@
 			)
 		)
-		(property "Description" "Polarized or Bipolar (C5-C7)"
+		(property "Description" "Polarized capacitor"
 			(at 238.252 29.718 90)
 			(effects
@@
 					(size 1.27 1.27)
 				)
+				(hide yes)
 			)
 		)

Commit message: Update PCB
Connections:
- net GND: now also J1.1 (S), J2.1 (S), J3.1 (S), J4.1 (S); no longer J1.2 (S), J2.2 (S), J3.2 (S), J4.2 (S)
- net at C1.2: now also J1.2 (T); no longer J1.1 (T)
- net at C7.2, R10.2: now also J4.2 (T); no longer J4.1 (T)
- net at C6.2, R9.2: now also J3.2 (T); no longer J3.1 (T)
- net at C5.2, R8.2: now also J2.2 (T); no longer J2.1 (T)

Commit message: Fix cap footprints
Parts:
- C1: footprint Capacitor_THT:C_Rect_L24.0mm_W7.0mm_P22.50mm_MKT -> Capacitor_THT:CP_Axial_L18.0mm_D8.0mm_P25.00mm_Horizontal
- C11, C9: footprint Capacitor_THT:C_Radial_D6.3mm_H11.0mm_P2.50mm -> Capacitor_THT:CP_Radial_D6.3mm_P2.50mm
- C5, C6, C7: footprint Capacitor_THT:C_Radial_D10.0mm_H12.5mm_P5.00mm -> Capacitor_THT:CP_Radial_D10.0mm_P5.00mm
Changed lines of the file:
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@@
 			)
 		)
-		(property "Footprint" "Capacitor_THT:C_Rect_L24.0mm_W7.0mm_P22.50mm_MKT"
+		(property "Footprint" "Capacitor_THT:CP_Axial_L18.0mm_D8.0mm_P25.00mm_Horizontal"
 			(at 46.99 42.8752 0)
 			(effects
@@
 			)
 		)
-		(property "Footprint" "Capacitor_THT:C_Radial_D6.3mm_H11.0mm_P2.50mm"
+		(property "Footprint" "Capacitor_THT:CP_Radial_D6.3mm_P2.50mm"
 			(at 102.5652 118.11 0)
 			(effects
@@
 			)
 		)
-		(property "Footprint" "Capacitor_THT:C_Radial_D6.3mm_H11.0mm_P2.50mm"
+		(property "Footprint" "Capacitor_THT:CP_Radial_D6.3mm_P2.50mm"
 			(at 64.4652 175.26 0)
 			(effects
@@
 			)
 		)
-		(property "Footprint" "Capacitor_THT:C_Radial_D10.0mm_H12.5mm_P5.00mm"
+		(property "Footprint" "Capacitor_THT:CP_Radial_D10.0mm_P5.00mm"
 			(at 238.76 106.9848 0)
 			(effects
@@
 			)
 		)
-		(property "Footprint" "Capacitor_THT:C_Radial_D10.0mm_H12.5mm_P5.00mm"
+		(property "Footprint" "Capacitor_THT:CP_Radial_D10.0mm_P5.00mm"
 			(at 238.76 43.4848 0)
 			(effects
@@
 			)
 		)
-		(property "Footprint" "Capacitor_THT:C_Radial_D10.0mm_H12.5mm_P5.00mm"
+		(property "Footprint" "Capacitor_THT:CP_Radial_D10.0mm_P5.00mm"
 			(at 238.76 75.2348 0)
 			(effects
